File: PowerBoard.kicad_pcb (KiCad board)
At the start: 2 copper layers, 150 x 150 mm, 132 parts, among them IC1 LT1910ES8#PBF, IC2 LT1910ES8#PBF, IC3 LT1910ES8#PBF, IC4 LT1910ES8#PBF, IC5 LT1910ES8#PBF, IC7 MAX17541GATB+T, J1 XT90, J10 XT90, J11 XT90, J12 XT90, J13 XT90, J14 DEAN_T, J15 DEAN_T, J16 DEAN_T, J17 DEAN_T, J18 DEAN_T, J19 DEAN_T, J2 DEAN_T, J20 XT60, J21 XT60, J22 XT60, J23 XT60, J24 XT60, J25 XT60, J26 XT60, J27 XT60, J28 XT60, J29 XT60, J3 XT60, J30 XT60, J31 XT60, J32 XT30, J33 XT30, J34 XT30, J35 XT30, J36 XT30, J37 XT30, J38 XT30, J39 XT30, J4 XT30, J40 XT30, J41 XT60, J5 Conn_01x02, J6 XT90, J7 XT90, J8 XT90, J9 XT90, Q1 IRFS7530TRL7PP, Q2 IRFS7437TRLPBF, Q3 IRFS7437TRLPBF, Q4 IRFS7437TRLPBF, Q5 IRFS7437TRLPBF, U1 Pico, U2 INA238, U3 INA238, U4 INA238, U5 INA238, U6 INA238

Commit message: v2.2.0
Routing:
- net SCL: track 125.6 -> 132.4 mm
- net GND: track 1201.6 -> 1206.8 mm
- net 12V_2: track 92.0 -> 95.3 mm
- net VCC: track 266.2 -> 269.2 mm
- net CURR_4+: track 53.0 -> 55.5 mm, vias 3 -> 2
- net CURR_5+: track 46.1 -> 48.6 mm
- net CURR_3+: track 79.6 -> 81.3 mm, vias 4 -> 2
- net CURR_4-: track 48.6 -> 50.3 mm
- net ALERT_3: track 126.6 -> 128.0 mm
- net ALERT_5: track 134.1 -> 135.1 mm
- net ALERT_4: track 134.5 -> 135.3 mm
- net ALERT_2: track 116.7 -> 117.4 mm
- net CURR_1+: track 61.6 -> 61.2 mm, vias 4 -> 2
- net CURR_2+: track 68.8 -> 69.1 mm, vias 4 -> 2
